File: hw/daisy_chain_board/daisy_chain_board.sch (KiCad schematic (older format))
At the start: 9 parts, among them J7 Conn_02x25_Odd_Even, J8 L717SDB25PA4CH4F, X1 Mac, X2 Dogcow, X3 Mac2, X4 Raspberry Pi, X7 Pi

Commit message: Cleanup LCSC part number, regenerate gerbers and re-generate schematics
Parts:
- J7: LCSC (none) -> C40024
- J8: value L717SDB25PA4CH4F -> CONFLY DB25; LCSC (none) -> C77838
Changed lines of the file:
@@
 F 2 "Connector_PinHeader_2.54mm:PinHeader_2x25_P2.54mm_Vertical" H 3550 2100 50  0001 C CNN
 F 3 "~" H 3550 2100 50  0001 C CNN
+F 4 "C40024" H 3550 2100 50  0001 C CNN "LCSC"
 	1    3550 2100
 	0    -1   -1   0
@@
 P 2900 2900
 F 0 "J8" V 2719 2900 50  0000 C CNN
-F 1 "L717SDB25PA4CH4F" V 2810 2900 50  0000 C CNN
+F 1 "CONFLY DB25" V 2810 2900 50  0000 C CNN
 F 2 "L717SDB25PA4CH4F" H 4550 3200 50  0001 L CNN
 F 3 "https://componentsearchengine.com/Datasheets/1/L717SDB25PA4CH4F.pdf" H 4550 3100 50  0001 L CNN
@@
 F 8 "Amphenol" H 4550 2600 50  0001 L CNN "Manufacturer_Name"
 F 9 "L717SDB25PA4CH4F" H 4550 2500 50  0001 L CNN "Manufacturer_Part_Number"
+F 10 "C77838" V 2900 2900 50  0001 C CNN "LCSC"
 	1    2900 2900
 	0    -1   1    0
