File: hw/rascsi_tester/rascsi_tester.kicad_pcb (KiCad board)
At the start: 2 copper layers, 65 x 56 mm, 92 parts, among them J1 USB_B_Micro, J2 Conn_02x25_Odd_Even, J3 Conn_01x02_Male, J4 L717SDB25PA4CH4F, X1 Mac, X2 Dogcow, X3 Mac2, X4 Raspberry Pi, X5 Dogcow2, X6 Mac Trashcan, X7 Pi, X8 Pi

Commit message: Updated tester board
Parts:
- removed X6: Mac Trashcan, SamacSys_Parts:mac_trashcan
- D1, D10, D11, D12, D13, D14, D15, D16, D17, D18, D19, D2, D3, D4, D5, D6, D7, D8, D9: footprint LED_SMD:LED_1206_3216Metric -> LED_SMD:LED_0805_2012Metric
- R1, R10, R11, R12, R13, R14, R15, R16, R17, R18, R19, R2, R3, R4, R5, R6, R7, R8, R9: footprint Resistor_SMD:R_1206_3216Metric_Pad1.42x1.75mm_HandSolder -> Resistor_SMD:R_0805_2012Metric
- X2: moved to B.Cu
- moved X7 41.4 mm to (236.5, 88.7)
- moved X8 40.0 mm to (222.0, 45.9)
- moved X3 39.5 mm to (216.5, 45.9)
- moved X5 27.1 mm to (187.5, 46.5)
- moved J3 19.7 mm to (195.5, 44.8)
- moved X4 12.2 mm to (227.9, 45.9)
- moved X2 11.4 mm to (188.2, 46.5), turned to 180 degrees
- moved J1 0.78 mm to (207.3, 44.6)
- moved JP33 0.06 mm to (207.0, 69.2)
Routing:
- net +5V: track 0.00 -> 137.7 mm, vias 0 -> 20
- net GND: track 56.9 -> 79.0 mm, vias 10 -> 21
- net Net-(D3-Pad2): track 0.00 -> 16.6 mm
- net Net-(D11-Pad2): track 0.00 -> 16.5 mm
- net Net-(D4-Pad2): track 0.00 -> 16.4 mm
- net Net-(D17-Pad2): track 0.00 -> 16.4 mm
- net Net-(D1-Pad2): track 0.00 -> 16.4 mm
- net Net-(D6-Pad2): track 0.00 -> 16.4 mm
- net Net-(D5-Pad2): track 0.00 -> 16.4 mm
- net Net-(D2-Pad2): track 0.00 -> 16.4 mm
- net Net-(D12-Pad2): track 0.00 -> 16.4 mm
- net Net-(D19-Pad2): track 0.00 -> 16.4 mm
- net Net-(D16-Pad2): track 0.00 -> 16.4 mm
- net Net-(D7-Pad2): track 0.00 -> 16.4 mm
- net Net-(D15-Pad2): track 0.00 -> 16.4 mm
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Other:
- board text added: "JLCJLCJLCJLC"
- board text added: "Test Board"
- board text removed: "10k"
- board text removed: "220"
- board text removed: "3.3"
- board text removed: "330"
- board text removed: "3v"
- board text removed: "ACT"
- board text removed: "ENB"
- board text removed: "FULLSPEC Board Version"
- board text removed: "GPIO0"
- board text removed: "GPIO1"
- board text removed: "GPIO9"
- board text removed: "J1"
- board text removed: "J4"
- board text removed: "J5"
- board text removed: "J7"
- board text removed: "J8"
- board text removed: "Only use the DB-25 OR 50-pin ribbon connector. DO NOT USE BOTH (Unless you REALLY know what you're doing)"
- board text removed: "SCL"
- board text removed: "SDA"
- board text removed: "Term Enable"
- board text removed: "USB Power"
